Commit message: Initial commit: UR3 MuJoCo simulation with MoveIt2 and RL bridge

File: src/Universal_Robots_ROS2_Driver/ur_moveit_config/srdf/ur_macro.srdf.xacro (robot description, xacro)
@@ -53,4 +53,25 @@
     <disable_collisions link1="${prefix}wrist_1_link" link2="${prefix}wrist_3_link" reason="Never" />
     <disable_collisions link1="${prefix}wrist_2_link" link2="${prefix}wrist_3_link" reason="Adjacent" />
+    <!-- MuJoCo table scene: mesh overlap between pedestal/base/cables and tabletop; props resting on table. -->
+    <disable_collisions link1="${prefix}base_link" link2="table" reason="Never" />
+    <disable_collisions link1="${prefix}base_link_inertia" link2="table" reason="Never" />
+    <disable_collisions link1="${prefix}shoulder_link" link2="table" reason="Never" />
+    <disable_collisions link1="${prefix}upper_arm_link" link2="table" reason="Never" />
+    <disable_collisions link1="sphere" link2="table" reason="Adjacent" />
+    <disable_collisions link1="cylinder" link2="table" reason="Adjacent" />
+    <disable_collisions link1="box" link2="table" reason="Adjacent" />
+    <!-- D435i / rl_camera TF tree vs adjacent UR links (visual mesh overlap; keep camera vs environment enabled). -->
+    <disable_collisions link1="${prefix}wrist_3_link" link2="d435i_mount_link" reason="Adjacent" />
+    <disable_collisions link1="${prefix}flange" link2="d435i_mount_link" reason="Adjacent" />
+    <disable_collisions link1="${prefix}tool0" link2="d435i_mount_link" reason="Adjacent" />
+    <disable_collisions link1="d435i_mount_link" link2="rl_camera_frame" reason="Adjacent" />
+    <disable_collisions link1="${prefix}flange" link2="rl_camera_frame" reason="Never" />
+    <disable_collisions link1="${prefix}tool0" link2="rl_camera_frame" reason="Never" />
+    <disable_collisions link1="${prefix}wrist_2_link" link2="d435i_mount_link" reason="Never" />
+    <disable_collisions link1="${prefix}wrist_1_link" link2="d435i_mount_link" reason="Never" />
+    <disable_collisions link1="${prefix}wrist_3_link" link2="rl_camera_frame" reason="Never" />
   </xacro:macro>
+  <disable_collisions link1="table" link2="sphere" reason="Adjacent" />
+  <disable_collisions link1="table" link2="cylinder" reason="Adjacent" />
+  <disable_collisions link1="table" link2="box" reason="Adjacent" />
 </robot>

File: src/ur3_mujoco_sim/urdf/ur3_mujoco_fixed.urdf.xacro (robot description, xacro)
@@ -39,4 +39,39 @@
   </xacro:ur_robot>
   <!--
+    D435i + rl_camera on wrist_3 (matches mjcf/UR3_RG2.xml: body d435i, camera pos 0 0 0.02, euler 0 -pi 0).
+    Cover mesh d435i_8 matches MuJoCo collision/visual shell. Optical frame for REP-103 / virtual_perception.
+  -->
+  <link name="d435i_mount_link"/>
+  <joint name="wrist_3_link_to_d435i_mount" type="fixed">
+    <parent link="wrist_3_link"/>
+    <child link="d435i_mount_link"/>
+    <origin xyz="0.02 0 0.05" rpy="0 1.5707963267948966 1.5707963267948966"/>
+  </joint>
+  <link name="rl_camera_frame">
+    <visual>
+      <origin xyz="0 0 0" rpy="0 0 0"/>
+      <geometry>
+        <mesh filename="package://ur3_mujoco_sim/meshes/d435i_8.obj" scale="1 1 1"/>
+      </geometry>
+    </visual>
+    <collision>
+      <origin xyz="0 0 0" rpy="0 0 0"/>
+      <geometry>
+        <mesh filename="package://ur3_mujoco_sim/meshes/d435i_8.obj" scale="1 1 1"/>
+      </geometry>
+    </collision>
+  </link>
+  <joint name="d435i_mount_to_rl_camera" type="fixed">
+    <parent link="d435i_mount_link"/>
+    <child link="rl_camera_frame"/>
+    <origin xyz="0 0 0.02" rpy="0 -3.141592653589793 0"/>
+  </joint>
+  <link name="camera_color_optical_frame"/>
+  <joint name="rl_camera_to_camera_color_optical" type="fixed">
+    <parent link="rl_camera_frame"/>
+    <child link="camera_color_optical_frame"/>
+    <origin xyz="0 0 0" rpy="-1.5707963267948966 0 -1.5707963267948966"/>
+  </joint>
+  <!--
     Scene props for RViz visualization.
     These mirror `mjcf/ur3_scene_table.xml` (same mesh files, same poses, no rotation).
@@ -61,23 +96,4 @@
     <origin xyz="0 0 0" rpy="0 0 0"/>
   </joint>
-  <link name="plate">
-    <visual>
-      <origin xyz="0 0 0" rpy="0 0 0"/>
-      <geometry>
-        <mesh filename="package://ur3_mujoco_sim/meshes/plate.stl" scale="0.001 0.001 0.001"/>
-      </geometry>
-    </visual>
-    <collision>
-      <origin xyz="0 0 0" rpy="0 0 0"/>
-      <geometry>
-        <mesh filename="package://ur3_mujoco_sim/meshes/plate.stl" scale="0.001 0.001 0.001"/>
-      </geometry>
-    </collision>
-  </link>
-  <joint name="world_to_plate" type="fixed">
-    <parent link="world"/>
-    <child link="plate"/>
-    <origin xyz="-0.3 0 0.4" rpy="0 0 0"/>
-  </joint>
   <link name="sphere">
     <visual>
@@ -98,23 +114,4 @@
     <child link="sphere"/>
     <origin xyz="-0.3 0.08 0.425" rpy="0 0 0"/>
-  </joint>
-  <link name="cup">
-    <visual>
-      <origin xyz="0 0 0" rpy="0 0 0"/>
-      <geometry>
-        <mesh filename="package://ur3_mujoco_sim/meshes/cup.stl" scale="0.001 0.001 0.001"/>
-      </geometry>
-    </visual>
-    <collision>
-      <origin xyz="0 0 0" rpy="0 0 0"/>
-      <geometry>
-        <mesh filename="package://ur3_mujoco_sim/meshes/cup.stl" scale="0.001 0.001 0.001"/>
-      </geometry>
-    </collision>
-  </link>
-  <joint name="world_to_cup" type="fixed">
-    <parent link="world"/>
-    <child link="cup"/>
-    <origin xyz="-0.3 0.16 0.4" rpy="0 0 0"/>
   </joint>
   <link name="cylinder">

Commit message: task 전

File: src/Universal_Robots_ROS2_Driver/ur_moveit_config/srdf/ur_macro.srdf.xacro (robot description, xacro)
@@ -62,5 +62,4 @@
     <disable_collisions link1="box" link2="table" reason="Adjacent" />
     <!-- D435i / rl_camera TF tree vs adjacent UR links (visual mesh overlap; keep camera vs environment enabled). -->
-    <disable_collisions link1="${prefix}wrist_3_link" link2="d435i_mount_link" reason="Adjacent" />
     <disable_collisions link1="${prefix}flange" link2="d435i_mount_link" reason="Adjacent" />
     <disable_collisions link1="${prefix}tool0" link2="d435i_mount_link" reason="Adjacent" />
@@ -71,7 +70,7 @@
     <disable_collisions link1="${prefix}wrist_1_link" link2="d435i_mount_link" reason="Never" />
     <disable_collisions link1="${prefix}wrist_3_link" link2="rl_camera_frame" reason="Never" />
+    <disable_collisions link1="table" link2="world" reason="Adjacent" />
+    <disable_collisions link1="table" link2="base_link_inertia" reason="Adjacent" />
+    <disable_collisions link1="table" link2="base_link" reason="Adjacent" />
   </xacro:macro>
-  <disable_collisions link1="table" link2="sphere" reason="Adjacent" />
-  <disable_collisions link1="table" link2="cylinder" reason="Adjacent" />
-  <disable_collisions link1="table" link2="box" reason="Adjacent" />
 </robot>

File: src/ur3_mujoco_sim/urdf/ur3_mujoco_fixed.urdf.xacro (robot description, xacro)
@@ -39,12 +39,13 @@
   </xacro:ur_robot>
   <!--
-    D435i + rl_camera on wrist_3 (matches mjcf/UR3_RG2.xml: body d435i, camera pos 0 0 0.02, euler 0 -pi 0).
-    Cover mesh d435i_8 matches MuJoCo collision/visual shell. Optical frame for REP-103 / virtual_perception.
+    D435i + rl_camera mounted on flange (same global pose as MJCF body d435i on link6_2_1; see UR3_RG2.xml).
+    Parent is flange — not wrist_3_link — so wrist_3_link keeps the standard UR subtree only (MoveIt/RViz).
+    Transform: inv(flange_from_wrist_3) * (old mount from wrist_3).
   -->
   <link name="d435i_mount_link"/>
-  <joint name="wrist_3_link_to_d435i_mount" type="fixed">
-    <parent link="wrist_3_link"/>
+  <joint name="flange_to_d435i_mount" type="fixed">
+    <parent link="$(arg tf_prefix)flange"/>
     <child link="d435i_mount_link"/>
-    <origin xyz="0.02 0 0.05" rpy="0 1.5707963267948966 1.5707963267948966"/>
+    <origin xyz="0.005 0 0.05" rpy="-1.5708 3.14159 1.5708"/>
   </joint>
   <link name="rl_camera_frame">

Commit message: 카메라 위치 수정 및 충돌 설정 업데이트

File: src/Universal_Robots_ROS2_Driver/ur_moveit_config/srdf/ur_macro.srdf.xacro (robot description, xacro)
@@ -56,21 +56,25 @@
     <disable_collisions link1="${prefix}base_link" link2="table" reason="Never" />
     <disable_collisions link1="${prefix}base_link_inertia" link2="table" reason="Never" />
-    <disable_collisions link1="${prefix}shoulder_link" link2="table" reason="Never" />
-    <disable_collisions link1="${prefix}upper_arm_link" link2="table" reason="Never" />
-    <disable_collisions link1="sphere" link2="table" reason="Adjacent" />
-    <disable_collisions link1="cylinder" link2="table" reason="Adjacent" />
-    <disable_collisions link1="box" link2="table" reason="Adjacent" />
     <!-- D435i / rl_camera TF tree vs adjacent UR links (visual mesh overlap; keep camera vs environment enabled). -->
-    <disable_collisions link1="${prefix}flange" link2="d435i_mount_link" reason="Adjacent" />
-    <disable_collisions link1="${prefix}tool0" link2="d435i_mount_link" reason="Adjacent" />
+    <!-- gripper/camera STL meshes overlap multiple wrist links → broad disables (matches tool0+wrist_* Never pattern above). -->
+    <disable_collisions link1="${prefix}tool0" link2="gripper_link" reason="Adjacent" />
+    <disable_collisions link1="${prefix}flange" link2="gripper_link" reason="Adjacent" />
+    <disable_collisions link1="${prefix}wrist_3_link" link2="gripper_link" reason="Adjacent" />
+    <disable_collisions link1="${prefix}wrist_2_link" link2="gripper_link" reason="Never" />
+    <disable_collisions link1="gripper_link" link2="d435i_mount_link" reason="Adjacent" />
     <disable_collisions link1="d435i_mount_link" link2="rl_camera_frame" reason="Adjacent" />
     <disable_collisions link1="${prefix}flange" link2="rl_camera_frame" reason="Never" />
     <disable_collisions link1="${prefix}tool0" link2="rl_camera_frame" reason="Never" />
+    <disable_collisions link1="${prefix}flange" link2="d435i_mount_link" reason="Adjacent" />
+    <disable_collisions link1="${prefix}tool0" link2="d435i_mount_link" reason="Adjacent" />
+    <disable_collisions link1="${prefix}wrist_3_link" link2="d435i_mount_link" reason="Adjacent" />
+    <disable_collisions link1="${prefix}wrist_2_link" link2="rl_camera_frame" reason="Never" />
+    <disable_collisions link1="${prefix}wrist_1_link" link2="rl_camera_frame" reason="Never" />
     <disable_collisions link1="${prefix}wrist_2_link" link2="d435i_mount_link" reason="Never" />
     <disable_collisions link1="${prefix}wrist_1_link" link2="d435i_mount_link" reason="Never" />
     <disable_collisions link1="${prefix}wrist_3_link" link2="rl_camera_frame" reason="Never" />
     <disable_collisions link1="table" link2="world" reason="Adjacent" />
-    <disable_collisions link1="table" link2="base_link_inertia" reason="Adjacent" />
-    <disable_collisions link1="table" link2="base_link" reason="Adjacent" />
+    <disable_collisions link1="table" link2="${prefix}base_link_inertia" reason="Adjacent" />
+    <disable_collisions link1="table" link2="${prefix}base_link" reason="Adjacent" />
   </xacro:macro>
 </robot>

File: src/ur3_mujoco_sim/urdf/ur3_mujoco_fixed.urdf.xacro (robot description, xacro)
@@ -36,16 +36,36 @@
     generate_ros2_control_tag="false"
     >
-    <origin xyz="0 0 0.4" rpy="0 0 -1.5708" />
+    <origin xyz="0 0 0.78" rpy="0 0 -1.5708" />
   </xacro:ur_robot>
   <!--
-    D435i + rl_camera mounted on flange (same global pose as MJCF body d435i on link6_2_1; see UR3_RG2.xml).
-    Parent is flange — not wrist_3_link — so wrist_3_link keeps the standard UR subtree only (MoveIt/RViz).
-    Transform: inv(flange_from_wrist_3) * (old mount from wrist_3).
+    gripper_test + D435i + rl_camera: matches MJCF UR3_RG2.xml (gripper_link on link6_2_1, d435i on gripper_link).
+    gripper_link is fixed to tool0 (same TCP as MJCF gripper body). Camera offset on gripper: pos 0.05 0 0.07, euler 0 1.57 1.57.
+    Mesh visual uses MJCF geom quat 0.5 0.5 0.5 0.5 → rpy 1.5708 0 1.5708 (fixed XYZ).
   -->
+  <link name="gripper_link">
+    <visual>
+      <origin xyz="0 0 0" rpy="1.5707963267948966 0 1.5707963267948966"/>
+      <geometry>
+        <mesh filename="package://ur3_mujoco_sim/meshes/gripper_test.stl" scale="0.001 0.001 0.001"/>
+      </geometry>
+    </visual>
+    <collision>
+      <origin xyz="0 0 0" rpy="1.5707963267948966 0 1.5707963267948966"/>
+      <geometry>
+        <mesh filename="package://ur3_mujoco_sim/meshes/gripper_test.stl" scale="0.001 0.001 0.001"/>
+      </geometry>
+    </collision>
+  </link>
+  <joint name="tool0_to_gripper_link" type="fixed">
+    <parent link="$(arg tf_prefix)tool0"/>
+    <child link="gripper_link"/>
+    <origin xyz="0 0 0" rpy="-1.5707963267948966 -1.5707963267948966 0"/>
+  </joint>
   <link name="d435i_mount_link"/>
-  <joint name="flange_to_d435i_mount" type="fixed">
-    <parent link="$(arg tf_prefix)flange"/>
+  <!-- Parent must be gripper_link so the chain matches MJCF (d435i is nested under gripper_link, not parallel to it). -->
+  <joint name="gripper_to_d435i_mount" type="fixed">
+    <parent link="gripper_link"/>
     <child link="d435i_mount_link"/>
-    <origin xyz="0.005 0 0.05" rpy="-1.5708 3.14159 1.5708"/>
+    <origin xyz="0.07 0 0.07" rpy="1.5707963267948966 0 -1.5707963267948966"/>
   </joint>
   <link name="rl_camera_frame">
@@ -80,13 +100,25 @@
   <link name="table">
     <visual>
-      <origin xyz="0 0 0" rpy="0 0 0"/>
+      <origin xyz="-0.441108 -0.28111 0" rpy="0 0 -1.5708"/>
       <geometry>
         <mesh filename="package://ur3_mujoco_sim/meshes/table.stl" scale="0.001 0.001 0.001"/>
       </geometry>
     </visual>
+    <visual>
+      <origin xyz="-0.441108 -0.28111 0.78" rpy="0 0 -1.5708"/>
+      <geometry>
+        <mesh filename="package://ur3_mujoco_sim/meshes/table_upper.stl" scale="0.001 0.001 0.001"/>
+      </geometry>
+    </visual>
     <collision>
-      <origin xyz="0 0 0" rpy="0 0 0"/>
+      <origin xyz="-0.441108 -0.28111 0" rpy="0 0 -1.5708"/>
       <geometry>
         <mesh filename="package://ur3_mujoco_sim/meshes/table.stl" scale="0.001 0.001 0.001"/>
+      </geometry>
+    </collision>
+    <collision>
+      <origin xyz="-0.441108 -0.28111 0.78" rpy="0 0 -1.5708"/>
+      <geometry>
+        <mesh filename="package://ur3_mujoco_sim/meshes/table_upper.stl" scale="0.001 0.001 0.001"/>
       </geometry>
     </collision>
@@ -96,61 +128,4 @@
     <child link="table"/>
     <origin xyz="0 0 0" rpy="0 0 0"/>
-  </joint>
-  <link name="sphere">
-    <visual>
-      <origin xyz="0 0 0" rpy="0 0 0"/>
-      <geometry>
-        <mesh filename="package://ur3_mujoco_sim/meshes/sphere.stl" scale="0.001 0.001 0.001"/>
-      </geometry>
-    </visual>
-    <collision>
-      <origin xyz="0 0 0" rpy="0 0 0"/>
-      <geometry>
-        <mesh filename="package://ur3_mujoco_sim/meshes/sphere.stl" scale="0.001 0.001 0.001"/>
-      </geometry>
-    </collision>
-  </link>
-  <joint name="world_to_sphere" type="fixed">
-    <parent link="world"/>
-    <child link="sphere"/>
-    <origin xyz="-0.3 0.08 0.425" rpy="0 0 0"/>
-  </joint>
-  <link name="cylinder">
-    <visual>
-      <origin xyz="0 0 0" rpy="0 0 0"/>
-      <geometry>
-        <mesh filename="package://ur3_mujoco_sim/meshes/cylinder.stl" scale="0.001 0.001 0.001"/>
-      </geometry>
-    </visual>
-    <collision>
-      <origin xyz="0 0 0" rpy="0 0 0"/>
-      <geometry>
-        <mesh filename="package://ur3_mujoco_sim/meshes/cylinder.stl" scale="0.001 0.001 0.001"/>
-      </geometry>
-    </collision>
-  </link>
-  <joint name="world_to_cylinder" type="fixed">
-    <parent link="world"/>
-    <child link="cylinder"/>
-    <origin xyz="-0.3 -0.08 0.4" rpy="0 0 0"/>
-  </joint>
-  <link name="box">
-    <visual>
-      <origin xyz="0 0 0" rpy="0 0 0"/>
-      <geometry>
-        <mesh filename="package://ur3_mujoco_sim/meshes/box.stl" scale="0.001 0.001 0.001"/>
-      </geometry>
-    </visual>
-    <collision>
-      <origin xyz="0 0 0" rpy="0 0 0"/>
-      <geometry>
-        <mesh filename="package://ur3_mujoco_sim/meshes/box.stl" scale="0.001 0.001 0.001"/>
-      </geometry>
-    </collision>
-  </link>
-  <joint name="world_to_box" type="fixed">
-    <parent link="world"/>
-    <child link="box"/>
-    <origin xyz="-0.3 -0.16 0.4" rpy="0 0 0"/>
   </joint>
   <!-- MuJoCo ros2_control system interface -->

Commit message: 카메라 위치 수정 및 충돌 설정 업데이트

File: src/Universal_Robots_ROS2_Driver/ur_moveit_config/srdf/ur_macro.srdf.xacro (robot description, xacro)
@@ -59,4 +59,6 @@
     <!-- gripper/camera STL meshes overlap multiple wrist links → broad disables (matches tool0+wrist_* Never pattern above). -->
     <disable_collisions link1="${prefix}tool0" link2="gripper_link" reason="Adjacent" />
+    <disable_collisions link1="${prefix}tool0" link2="gripper_tip" reason="Adjacent" />
+    <disable_collisions link1="gripper_link" link2="gripper_tip" reason="Adjacent" />
     <disable_collisions link1="${prefix}flange" link2="gripper_link" reason="Adjacent" />
     <disable_collisions link1="${prefix}wrist_3_link" link2="gripper_link" reason="Adjacent" />

File: src/ur3_mujoco_sim/urdf/ur3_mujoco_fixed.urdf.xacro (robot description, xacro)
@@ -25,4 +25,44 @@
   <xacro:arg name="camera_depth_dropout_prob" default="0.0"/>
   <xacro:arg name="lidar_publish_rate" default="5.0"/>
+  <!-- Visual-only RGB axis marker (no collision). -->
+  <xacro:macro name="axis_marker_link" params="name parent xyz:='0 0 0' rpy:='0 0 0' length:='0.05' radius:='0.0025'">
+    <link name="${name}">
+      <!-- +X axis (red) -->
+      <visual>
+        <origin xyz="${length*0.5} 0 0" rpy="0 1.5707963267948966 0"/>
+        <geometry>
+          <cylinder length="${length}" radius="${radius}"/>
+        </geometry>
+        <material name="${name}_x_red">
+          <color rgba="1 0 0 1"/>
+        </material>
+      </visual>
+      <!-- +Y axis (green) -->
+      <visual>
+        <origin xyz="0 ${length*0.5} 0" rpy="-1.5707963267948966 0 0"/>
+        <geometry>
+          <cylinder length="${length}" radius="${radius}"/>
+        </geometry>
+        <material name="${name}_y_green">
+          <color rgba="0 1 0 1"/>
+        </material>
+      </visual>
+      <!-- +Z axis (blue) -->
+      <visual>
+        <origin xyz="0 0 ${length*0.5}" rpy="0 0 0"/>
+        <geometry>
+          <cylinder length="${length}" radius="${radius}"/>
+        </geometry>
+        <material name="${name}_z_blue">
+          <color rgba="0 0 1 1"/>
+        </material>
+      </visual>
+    </link>
+    <joint name="${name}_joint" type="fixed">
+      <parent link="${parent}"/>
+      <child link="${name}"/>
+      <origin xyz="${xyz}" rpy="${rpy}"/>
+    </joint>
+  </xacro:macro>
   <!-- Official UR model macros -->
   <xacro:include filename="$(find ur_description)/urdf/ur_macro.xacro"/>
@@ -40,4 +80,5 @@
     generate_ros2_control_tag="false"
     >
+    <!-- Align URDF world frame with MuJoCo world frame (no extra yaw offset). -->
     <origin xyz="0 0 0.78" rpy="0 0 -1.5707963267948966" />
   </xacro:ur_robot>
@@ -48,4 +89,9 @@
   -->
   <link name="gripper_link">
+  <inertial>
+      <origin xyz="0 0 0.05" rpy="0 0 0"/>
+      <mass value="0.5"/>
+      <inertia ixx="0.001" ixy="0" ixz="0" iyy="0.001" iyz="0" izz="0.001"/>
+  </inertial>
     <visual>
       <origin xyz="0 0 0" rpy="0 0 0"/>
@@ -65,4 +111,14 @@
     <child link="gripper_link"/>
     <origin xyz="0 0 0" rpy="0 0 0"/>
+  </joint>
+  <!--
+    TCP used by ur3_pick_task / MoveIt IK (must match ur3_rl_bridge/config/tcp/gripper_tip.yaml).
+    Visual-only: empty link + axis marker for RViz; same offset as YAML tool0 -> gripper_tip.
+  -->
+  <link name="gripper_tip"/>
+  <joint name="tool0_to_gripper_tip" type="fixed">
+    <parent link="$(arg tf_prefix)tool0"/>
+    <child link="gripper_tip"/>
+    <origin xyz="0 0 0.14" rpy="0 0 0"/>
   </joint>
   <link name="d435i_mount_link"/>
@@ -98,4 +154,14 @@
     <origin xyz="0 0 0" rpy="0 0 0"/>
   </joint>
+  <!-- Axis markers on major UR frames (visual-only, no collisions). -->
+  <xacro:axis_marker_link name="$(arg tf_prefix)axis_base_link" parent="$(arg tf_prefix)base_link" length="0.06" radius="0.0025"/>
+  <xacro:axis_marker_link name="$(arg tf_prefix)axis_shoulder_link" parent="$(arg tf_prefix)shoulder_link" length="0.05" radius="0.0022"/>
+  <xacro:axis_marker_link name="$(arg tf_prefix)axis_upper_arm_link" parent="$(arg tf_prefix)upper_arm_link" length="0.05" radius="0.0022"/>
+  <xacro:axis_marker_link name="$(arg tf_prefix)axis_forearm_link" parent="$(arg tf_prefix)forearm_link" length="0.05" radius="0.0022"/>
+  <xacro:axis_marker_link name="$(arg tf_prefix)axis_wrist_1_link" parent="$(arg tf_prefix)wrist_1_link" length="0.04" radius="0.002"/>
+  <xacro:axis_marker_link name="$(arg tf_prefix)axis_wrist_2_link" parent="$(arg tf_prefix)wrist_2_link" length="0.04" radius="0.002"/>
+  <xacro:axis_marker_link name="$(arg tf_prefix)axis_wrist_3_link" parent="$(arg tf_prefix)wrist_3_link" length="0.04" radius="0.002"/>
+  <xacro:axis_marker_link name="$(arg tf_prefix)axis_tool0" parent="$(arg tf_prefix)tool0" length="0.04" radius="0.002"/>
+  <xacro:axis_marker_link name="$(arg tf_prefix)axis_gripper_tip" parent="gripper_tip" length="0.07" radius="0.0025"/>
   <!--
     Scene props for RViz visualization.
