Commit message: Add real-robot FoundationPose grasp pipeline and pick sequence updates.
FoundationPose on RealSense, YOLO seg masks, stable fp_object TF, base_link
grip offsets, two-stage hover/plunge grasp, and expanded real/sim action YAML.

Co-authored-by: Cursor <cursoragent@cursor.com>

File: src/Universal_Robots_ROS2_Driver/ur_moveit_config/srdf/ur_macro.srdf.xacro (robot description, xacro)
@@ -76,4 +76,5 @@
     <disable_collisions link1="${prefix}wrist_1_link" link2="d435i_mount_link" reason="Never" />
     <disable_collisions link1="${prefix}wrist_3_link" link2="rl_camera_frame" reason="Never" />
+    <disable_collisions link1="rl_camera_jack" link2="rl_camera_frame" reason="Never" />
     <disable_collisions link1="table" link2="world" reason="Adjacent" />
     <disable_collisions link1="table" link2="${prefix}base_link_inertia" reason="Adjacent" />

File: src/ur3_mujoco_sim/urdf/ur3_mujoco_fixed.urdf.xacro (robot description, xacro)
@@ -144,5 +144,5 @@
     <parent link="$(arg tf_prefix)tool0"/>
     <child link="gripper_tip"/>
-    <origin xyz="0 0 0.14" rpy="0 0 0"/>
+    <origin xyz="0 0 0.146136" rpy="0 0 0"/>
   </joint>
   <link name="d435i_mount_link"/>
