Commit message: 카메라 위치 수정 및 충돌 설정 업데이트

File: src/ur3_mujoco_sim/urdf/ur3_mujoco_fixed.urdf.xacro (robot description, xacro)
@@ -20,4 +20,8 @@
   <xacro:arg name="headless" default="false"/>
   <xacro:arg name="camera_publish_rate" default="5.0"/>
+  <xacro:arg name="camera_rgb_noise_sigma" default="0.0"/>
+  <xacro:arg name="camera_depth_noise_sigma_m" default="0.0"/>
+  <xacro:arg name="camera_depth_quant_step_m" default="0.0"/>
+  <xacro:arg name="camera_depth_dropout_prob" default="0.0"/>
   <xacro:arg name="lidar_publish_rate" default="5.0"/>
   <!-- Official UR model macros -->
@@ -36,5 +40,5 @@
     generate_ros2_control_tag="false"
     >
-    <origin xyz="0 0 0.78" rpy="0 0 -1.5708" />
+    <origin xyz="0 0 0.78" rpy="0 0 -1.5707963267948966" />
   </xacro:ur_robot>
   <!--
@@ -45,5 +49,5 @@
   <link name="gripper_link">
     <visual>
-      <origin xyz="0 0 0" rpy="1.5707963267948966 0 1.5707963267948966"/>
+      <origin xyz="0 0 0" rpy="0 0 0"/>
       <geometry>
         <mesh filename="package://ur3_mujoco_sim/meshes/gripper_test.stl" scale="0.001 0.001 0.001"/>
@@ -51,5 +55,5 @@
     </visual>
     <collision>
-      <origin xyz="0 0 0" rpy="1.5707963267948966 0 1.5707963267948966"/>
+      <origin xyz="0 0 0" rpy="0 0 0"/>
       <geometry>
         <mesh filename="package://ur3_mujoco_sim/meshes/gripper_test.stl" scale="0.001 0.001 0.001"/>
@@ -60,5 +64,5 @@
     <parent link="$(arg tf_prefix)tool0"/>
     <child link="gripper_link"/>
-    <origin xyz="0 0 0" rpy="-1.5707963267948966 -1.5707963267948966 0"/>
+    <origin xyz="0 0 0" rpy="0 0 0"/>
   </joint>
   <link name="d435i_mount_link"/>
@@ -67,17 +71,17 @@
     <parent link="gripper_link"/>
     <child link="d435i_mount_link"/>
-    <origin xyz="0.07 0 0.07" rpy="1.5707963267948966 0 -1.5707963267948966"/>
+    <origin xyz="0 0.07 0.05" rpy="0 0 0"/>
   </joint>
   <link name="rl_camera_frame">
     <visual>
-      <origin xyz="0 0 0" rpy="0 0 0"/>
+      <origin xyz="0.0325 0 0" rpy="0 0 0"/>
       <geometry>
-        <mesh filename="package://ur3_mujoco_sim/meshes/d435i_8.obj" scale="1 1 1"/>
+        <mesh filename="package://ur3_mujoco_sim/meshes/d435i_8.obj" scale="0.1 0.1 0.1"/>
       </geometry>
     </visual>
     <collision>
-      <origin xyz="0 0 0" rpy="0 0 0"/>
+      <origin xyz="0.0325 0 0" rpy="0 0 0"/>
       <geometry>
-        <mesh filename="package://ur3_mujoco_sim/meshes/d435i_8.obj" scale="1 1 1"/>
+        <mesh filename="package://ur3_mujoco_sim/meshes/d435i_8.obj" scale="0.1 0.1 0.1"/>
       </geometry>
     </collision>
@@ -86,5 +90,5 @@
     <parent link="d435i_mount_link"/>
     <child link="rl_camera_frame"/>
-    <origin xyz="0 0 0.02" rpy="0 -3.141592653589793 0"/>
+    <origin xyz="0 0 0" rpy="0 0 0"/>
   </joint>
   <link name="camera_color_optical_frame"/>
@@ -92,5 +96,5 @@
     <parent link="rl_camera_frame"/>
     <child link="camera_color_optical_frame"/>
-    <origin xyz="0 0 0" rpy="-1.5707963267948966 0 -1.5707963267948966"/>
+    <origin xyz="0 0 0" rpy="0 0 0"/>
   </joint>
   <!--
@@ -137,4 +141,8 @@
       <param name="headless">$(arg headless)</param>
       <param name="camera_publish_rate">$(arg camera_publish_rate)</param>
+      <param name="camera_rgb_noise_sigma">$(arg camera_rgb_noise_sigma)</param>
+      <param name="camera_depth_noise_sigma_m">$(arg camera_depth_noise_sigma_m)</param>
+      <param name="camera_depth_quant_step_m">$(arg camera_depth_quant_step_m)</param>
+      <param name="camera_depth_dropout_prob">$(arg camera_depth_dropout_prob)</param>
       <param name="lidar_publish_rate">$(arg lidar_publish_rate)</param>
     </hardware>

Commit message: 카메라 위치 수정 및 충돌 설정 업데이트

File: src/ur3_mujoco_sim/urdf/ur3_mujoco_fixed.urdf.xacro (robot description, xacro)
@@ -154,4 +154,22 @@
     <origin xyz="0 0 0" rpy="0 0 0"/>
   </joint>
+  <!--
+    MuJoCo-only gripper actuator DOF (MJCF joint name must match): no meshes — a virtual link for ros2_control + joint_states.
+    Physics/visual gripper stays in MJCF (UR3_RG2.xml); RViz shows no extra geometry. Use gripper_motor_position_controller to command.
+  -->
+  <link name="gripper_motor_dummy">
+    <inertial>
+      <origin xyz="0 0 0" rpy="0 0 0"/>
+      <mass value="0.001"/>
+      <inertia ixx="1e-9" ixy="0" ixz="0" iyy="1e-9" iyz="0" izz="1e-9"/>
+    </inertial>
+  </link>
+  <joint name="$(arg tf_prefix)gripper_motor_joint" type="revolute">
+    <parent link="$(arg tf_prefix)tool0"/>
+    <child link="gripper_motor_dummy"/>
+    <origin xyz="0 0 0" rpy="0 0 0"/>
+    <axis xyz="0 0 1"/>
+    <limit lower="0" upper="1.396" effort="10" velocity="2"/>
+  </joint>
   <!-- Axis markers on major UR frames (visual-only, no collisions). -->
   <xacro:axis_marker_link name="$(arg tf_prefix)axis_base_link" parent="$(arg tf_prefix)base_link" length="0.06" radius="0.0025"/>
@@ -243,4 +261,9 @@
       <state_interface name="velocity"/>
     </joint>
+    <joint name="$(arg tf_prefix)gripper_motor_joint">
+      <command_interface name="position"/>
+      <state_interface name="position"/>
+      <state_interface name="velocity"/>
+    </joint>
   </ros2_control>
 </robot>

Commit message: 카메라 위치 수정 및 충돌 설정 업데이트

File: src/ur3_mujoco_sim/urdf/ur3_mujoco_fixed.urdf.xacro (robot description, xacro)
@@ -95,13 +95,37 @@
   </inertial>
     <visual>
-      <origin xyz="0 0 0" rpy="0 0 0"/>
-      <geometry>
-        <mesh filename="package://ur3_mujoco_sim/meshes/gripper_test.stl" scale="0.001 0.001 0.001"/>
-      </geometry>
-    </visual>
-    <collision>
-      <origin xyz="0 0 0" rpy="0 0 0"/>
-      <geometry>
-        <mesh filename="package://ur3_mujoco_sim/meshes/gripper_test.stl" scale="0.001 0.001 0.001"/>
+      <origin xyz="0 0 0" rpy="3.14159262 0 -1.57"/>
+      <geometry>
+        <mesh filename="package://ur3_mujoco_sim/meshes/gripper/Case_Base.stl" scale="0.001 0.001 0.001"/>
+      </geometry>
+    </visual>
+    <collision>
+      <origin xyz="0 0 0" rpy="3.14159262 0 -1.57"/>
+      <geometry>
+        <mesh filename="package://ur3_mujoco_sim/meshes/gripper/Case_Base.stl" scale="0.001 0.001 0.001"/>
+      </geometry>
+    </collision>
+    <visual>
+      <origin xyz="0 0 0" rpy="3.14159262 0 -1.57"/>
+      <geometry>
+        <mesh filename="package://ur3_mujoco_sim/meshes/gripper/Case_Latch.stl" scale="0.001 0.001 0.001"/>
+      </geometry>
+    </visual>
+    <collision>
+      <origin xyz="0 0 0" rpy="3.14159262 0 -1.57"/>
+      <geometry>
+        <mesh filename="package://ur3_mujoco_sim/meshes/gripper/Case_Latch.stl" scale="0.001 0.001 0.001"/>
+      </geometry>
+    </collision>
+    <visual>
+      <origin xyz="0 0 0" rpy="3.14159262 0 -1.57"/>
+      <geometry>
+        <mesh filename="package://ur3_mujoco_sim/meshes/gripper/Shaft.stl" scale="0.001 0.001 0.001"/>
+      </geometry>
+    </visual>
+    <collision>
+      <origin xyz="0 0 0" rpy="3.14159262 0 -1.57"/>
+      <geometry>
+        <mesh filename="package://ur3_mujoco_sim/meshes/gripper/Shaft.stl" scale="0.001 0.001 0.001"/>
       </geometry>
     </collision>
@@ -131,5 +155,5 @@
   <link name="rl_camera_frame">
     <visual>
-      <origin xyz="0.0325 0 0" rpy="0 0 0"/>
+      <origin xyz="0 0 0" rpy="0 0 0"/>
       <geometry>
         <mesh filename="package://ur3_mujoco_sim/meshes/d435i_8.obj" scale="0.1 0.1 0.1"/>
@@ -137,5 +161,5 @@
     </visual>
     <collision>
-      <origin xyz="0.0325 0 0" rpy="0 0 0"/>
+      <origin xyz="0 0 0" rpy="0 0 0"/>
       <geometry>
         <mesh filename="package://ur3_mujoco_sim/meshes/d435i_8.obj" scale="0.1 0.1 0.1"/>
@@ -146,11 +170,12 @@
     <parent link="d435i_mount_link"/>
     <child link="rl_camera_frame"/>
-    <origin xyz="0 0 0" rpy="0 0 0"/>
-  </joint>
+    <origin xyz="0.0325 0 0" rpy="0 0 0"/>
+  </joint>
+  <!-- REP-103 optical frame: Z into scene (+depth), X right, Y down in image. MuJoCo rl_camera uses euler 0 -π 0 on d435i body. -->
   <link name="camera_color_optical_frame"/>
   <joint name="rl_camera_to_camera_color_optical" type="fixed">
     <parent link="rl_camera_frame"/>
     <child link="camera_color_optical_frame"/>
-    <origin xyz="0 0 0" rpy="0 0 0"/>
+    <origin xyz="0 0 0" rpy="0 0 -3.141592653589793"/>
   </joint>
   <!--
@@ -266,4 +291,11 @@
       <state_interface name="velocity"/>
     </joint>
+    <!-- Sensor name must match MJCF camera name (rl_camera). Images/depth use optical frame (matches MJCF camera euler). -->
+    <sensor name="rl_camera">
+      <param name="frame_name">camera_color_optical_frame</param>
+      <param name="info_topic">/rl_camera/camera_info</param>
+      <param name="image_topic">/rl_camera/color</param>
+      <param name="depth_topic">/rl_camera/depth</param>
+    </sensor>
   </ros2_control>
 </robot>
